File: Electrical-Design/MPPT-Charge-Controller-KiCad/MPPT Charge Controller.kicad_sch (KiCad schematic)
At the start: 57 parts, among them Q1 SI7272DP, Q3 2N7002, U2 AP63203WU, U3 ACS712, U4 ACS712, U5 MCP4018

Commit message: Update schematics - delete tracks - 4 layer boards have only 2 signal layers
Parts:
- C1, C16, C18: footprint Capacitor_SMD:C_1210_3225Metric -> Capacitor_SMD:C_0603_1608Metric
- C17, C19: value 100nF -> 0.1uF; footprint Capacitor_SMD:C_1210_3225Metric -> Capacitor_SMD:C_0603_1608Metric
- C9: footprint Capacitor_SMD:C_0805_2012Metric -> Capacitor_SMD:C_0603_1608Metric
- M2: footprint MegaCastle:MegaCastle2x23-Module-I30.0x53.6-M80000307FFFC-PANEL -> MPPT Charge Controller Footprint Library:MegaCastle2x24-Module-I40.0x56.2-M8000030FFFFF-SPAREPAD; symbol MegaCastle:MegaCastle2x23-Module-I30.0x53.6-M80000307FFFC -> MPPT-Charge-Controller-Controller:MegaCastle2x24-Module-I40.0x56.2-M8000030FFFFF
Connections:
- net +3.3V: now also M2.43; no longer M2.41
- net BTST: now also M2.35; no longer M2.33
- net GND: now also C15.2, C2.2, C3.2, M2.24 (GND), M2.46, NT1.1, NT2.1, NT3.1, NT4.1, Q3.2 (S), R1.2, R10.2, R4.2, U1.11 (GND), U1.17 (Thermal_Pad), U5.2 (VSS); no longer M2.23 (GND)
- net HIDRV: now also M2.34; no longer M2.32
- net Input: now also M2.29; no longer M2.24
- net LODRV: now also M2.33; no longer M2.31
- net MPPSET: now also M2.41; no longer M2.39
- net PH: now also M2.32; no longer M2.30
- net RGEN: now also M2.36; no longer M2.34
- net SD_CS: now also M2.31
- net STAT1: now also M2.45; no longer M2.43
- net STAT2: now also M2.44; no longer M2.42
- net TS: now also M2.40; no longer M2.38
- net UART_RX: now also M2.48; no longer M2.46
- net UART_TX: now also M2.47; no longer M2.45
- net VCC: now also M2.37; no longer M2.35
- net VFB: now also M2.39; no longer M2.37
- net VREF: now also M2.38; no longer M2.36
- net ~{Charge EN}: now also M2.42; no longer M2.40
- removed net PWR GND: C15.2, C2.2, C3.2, M2.44, NT1.1, NT2.1, NT3.1, NT4.1, Q3.2 (S), R1.2, R10.2, R4.2, U1.11 (GND), U1.17 (Thermal_Pad), U5.2 (VSS)
Other:
- moved on the sheet: Q3
